Commit message: WIP
Added depth cam

File: sawyer_description/urdf/sawyer.urdf.xacro (robot description, xacro)
@@ -2,7 +2,8 @@
 <robot name="sawyer" xmlns:xacro="http://www.ros.org/wiki/xacro">
   <xacro:arg name="gazebo" default="false"/>
-  <xacro:arg name="pedestal" default="true"/>
+  <xacro:arg name="pedestal" default="false"/>
   <xacro:arg name="static" default="true"/>
   <xacro:arg name="electric_gripper" default="false"/>
+  <xacro:arg name="camera" default="true"/>
   <!-- Sawyer Base URDF -->
   <xacro:include filename="$(find sawyer_description)/urdf/sawyer_base.urdf.xacro">
@@ -22,3 +23,10 @@
   </xacro:include>
   </xacro:if>
+  <!-- Depth Camera -->
+  <xacro:if value="$(arg camera)">
+  <xacro:include filename="$(find realsense2_description)/urdf/_d435.urdf.xacro"/>
+  <xacro:sensor_d435 name="camera" parent="right_hand" use_nominal_extrinsics="true">
+    <origin xyz="0 -0.075 0.09" rpy="0 ${-pi/2} ${pi/2}"/>
+  </xacro:sensor_d435>
+  </xacro:if>
 </robot>
